File: docs/KiCad/ESP_Steckdose/ESP_Steckdose.sch (KiCad schematic (older format))
At the start: 32 parts, among them J1 Conn_01x03_Female, J2 Conn_01x03_Female, J3 Conn_01x03_Female, J4 Conn_01x03_Female, J5 Conn_01x03_Female, K1 G5V-1, K2 G5V-1, K3 G5V-1, K4 G5V-1, K5 G5V-1

Commit message: Utils update
Parts:
- R1, R2, R3, R4, R5: renamed from R?; value R -> 2.2k
- R10, R9: renamed from R?; value R -> 100
- R6, R7, R8: renamed from R?; value R -> 220
- gave numbers to parts that had none: 2
Changed lines of the file:
@@
 $EndDescr
 $Comp
-L MCU_Module:WeMos_D1_mini U?
+L MCU_Module:WeMos_D1_mini U1
 U 1 1 63FB08E9
 P 1200 2700
-F 0 "U?" H 1200 1811 50  0000 C CNN
-F 1 "WeMos_D1_mini" H 1200 1720 50  0000 C CNN
+F 0 "U1" H 1550 1850 50  0000 C CNN
+F 1 "WeMos_D1_mini" H 1550 1950 50  0000 C CNN
 F 2 "Module:WEMOS_D1_mini_light" H 1200 1550 50  0001 C CNN
 F 3 "https://wiki.wemos.cc/products:d1:d1_mini#documentation" H -650 1550 50  0001 C CNN
@@
 $EndComp
 $Comp
-L 74xx:74AHC595 U?
+L 74xx:74AHC595 U2
 U 1 1 63FB1383
 P 3600 1450
-F 0 "U?" H 3600 2231 50  0000 C CNN
-F 1 "74AHC595" H 3600 2140 50  0000 C CNN
+F 0 "U2" H 3850 2100 50  0000 C CNN
+F 1 "74AHC595" H 3850 2000 50  0000 C CNN
 F 2 "" H 3600 1450 50  0001 C CNN
 F 3 "https://assets.nexperia.com/documents/data-sheet/74AHC_AHCT595.pdf" H 3600 1450 50  0001 C CNN
@@
 	4850 5600 8150 5600
 $Comp
-L Device:R R?
+L Device:R R5
 U 1 1 6407EC7C
 P 5700 6400
-F 0 "R?" H 5770 6446 50  0000 L CNN
-F 1 "R" H 5770 6355 50  0000 L CNN
+F 0 "R5" H 5770 6446 50  0000 L CNN
+F 1 "2.2k" H 5770 6355 50  0000 L CNN
 F 2 "" V 5630 6400 50  0001 C CNN
 F 3 "~" H 5700 6400 50  0001 C CNN
@@
 $EndComp
 $Comp
-L Device:R R?
+L Device:R R10
 U 1 1 64080476
 P 6900 6200
-F 0 "R?" H 6970 6246 50  0000 L CNN
-F 1 "R" H 6970 6155 50  0000 L CNN
+F 0 "R10" H 6970 6246 50  0000 L CNN
+F 1 "100" H 6970 6155 50  0000 L CNN
 F 2 "" V 6830 6200 50  0001 C CNN
 F 3 "~" H 6900 6200 50  0001 C CNN
@@
 $EndComp
 $Comp
-L Device:R R?
+L Device:R R9
 U 1 1 640819E5
 P 6850 5050
-F 0 "R?" H 6920 5096 50  0000 L CNN
-F 1 "R" H 6920 5005 50  0000 L CNN
+F 0 "R9" H 6920 5096 50  0000 L CNN
+F 1 "100" H 6920 5005 50  0000 L CNN
 F 2 "" V 6780 5050 50  0001 C CNN
 F 3 "~" H 6850 5050 50  0001 C CNN
@@
 $EndComp
 $Comp
-L Device:R R?
+L Device:R R8
 U 1 1 64082E00
 P 6850 4000
-F 0 "R?" H 6920 4046 50  0000 L CNN
-F 1 "R" H 6920 3955 50  0000 L CNN
+F 0 "R8" H 6920 4046 50  0000 L CNN
+F 1 "220" H 6920 3955 50  0000 L CNN
 F 2 "" V 6780 4000 50  0001 C CNN
 F 3 "~" H 6850 4000 50  0001 C CNN
@@
 $EndComp
 $Comp
-L Device:R R?
+L Device:R R7
 U 1 1 6408425A
 P 6850 2850
-F 0 "R?" H 6920 2896 50  0000 L CNN
-F 1 "R" H 6920 2805 50  0000 L CNN
+F 0 "R7" H 6920 2896 50  0000 L CNN
+F 1 "220" H 6920 2805 50  0000 L CNN
 F 2 "" V 6780 2850 50  0001 C CNN
 F 3 "~" H 6850 2850 50  0001 C CNN
@@
 $EndComp
 $Comp
-L Device:R R?
-U 1 1 64086B8C
-P 5700 2050
-F 0 "R?" H 5770 2096 50  0000 L CNN
-F 1 "R" H 5770 2005 50  0000 L CNN
-F 2 "" V 5630 2050 50  0001 C CNN
-F 3 "~" H 5700 2050 50  0001 C CNN
-	1    5700 2050
-	0    -1   -1   0
-$EndComp
-$Comp
-L Device:R R?
+L Device:R R2
 U 1 1 64088194
 P 5700 3050
-F 0 "R?" H 5770 3096 50  0000 L CNN
-F 1 "R" H 5770 3005 50  0000 L CNN
+F 0 "R2" H 5770 3096 50  0000 L CNN
+F 1 "2.2k" H 5770 3005 50  0000 L CNN
 F 2 "" V 5630 3050 50  0001 C CNN
 F 3 "~" H 5700 3050 50  0001 C CNN
@@
 $EndComp
 $Comp
-L Device:R R?
+L Device:R R3
 U 1 1 640897B0
 P 5700 4200
-F 0 "R?" H 5770 4246 50  0000 L CNN
-F 1 "R" H 5770 4155 50  0000 L CNN
+F 0 "R3" H 5770 4246 50  0000 L CNN
+F 1 "2.2k" H 5770 4155 50  0000 L CNN
 F 2 "" V 5630 4200 50  0001 C CNN
 F 3 "~" H 5700 4200 50  0001 C CNN
@@
 $EndComp
 $Comp
-L Device:R R?
+L Device:R R4
 U 1 1 6408ADB1
 P 5700 5250
-F 0 "R?" H 5770 5296 50  0000 L CNN
-F 1 "R" H 5770 5205 50  0000 L CNN
+F 0 "R4" H 5770 5296 50  0000 L CNN
+F 1 "2.2k" H 5770 5205 50  0000 L CNN
 F 2 "" V 5630 5250 50  0001 C CNN
 F 3 "~" H 5700 5250 50  0001 C CNN
@@
 	6450 1850 6650 1850
 $Comp
-L Device:R R?
+L Device:R R6
 U 1 1 640856C9
 P 6800 1850
-F 0 "R?" H 6870 1896 50  0000 L CNN
-F 1 "R" H 6870 1805 50  0000 L CNN
+F 0 "R6" H 6870 1896 50  0000 L CNN
+F 1 "220" H 6870 1805 50  0000 L CNN
 F 2 "" V 6730 1850 50  0001 C CNN
 F 3 "~" H 6800 1850 50  0001 C CNN
@@
 	-1   0    0    1
 $EndComp
+$Comp
+L Device:R R1
+U 1 1 64086B8C
+P 5700 2050
+F 0 "R1" H 5750 2100 50  0000 L CNN
+F 1 "2.2k" H 5750 2000 50  0000 L CNN
+F 2 "" V 5630 2050 50  0001 C CNN
+F 3 "~" H 5700 2050 50  0001 C CNN
+	1    5700 2050
+	0    -1   -1   0
+$EndComp
 $EndSCHEMATC

Commit message: corect plan
Connections:
- wire segments 148 -> 150
Changed lines of the file:
@@
 NoConn ~ 6050 6200
 Wire Wire Line
-	1600 2600 4650 2600
-Wire Wire Line
-	4650 2600 4650 1650
-Wire Wire Line
-	4650 1650 6050 1650
-Wire Wire Line
-	6050 2700 6050 2650
-Wire Wire Line
-	1600 2700 6050 2700
+	4650 2650 6050 2650
 Wire Wire Line
 	1600 2800 4650 2800
@@
 	0    -1   -1   0
 $EndComp
+$Comp
+L power:GND #PWR?
+U 1 1 63FADA4F
+P 7500 6300
+F 0 "#PWR?" H 7500 6050 50  0001 C CNN
+F 1 "GND" H 7505 6127 50  0000 C CNN
+F 2 "" H 7500 6300 50  0001 C CNN
+F 3 "" H 7500 6300 50  0001 C CNN
+	1    7500 6300
+	1    0    0    -1
+$EndComp
+Wire Wire Line
+	7500 6300 7500 6200
+Wire Wire Line
+	4650 2650 4650 2700
+Wire Wire Line
+	4650 2700 1600 2700
+Wire Wire Line
+	4550 1650 4550 2600
+Wire Wire Line
+	4550 2600 1600 2600
+Wire Wire Line
+	4550 1650 6050 1650
 $EndSCHEMATC

Commit message: Änderung Plan
Connections:
- wire segments 150 -> 151
- no-connect marks 21 -> 20
Other:
- moved on the sheet: U1
Changed lines of the file:
@@
 L MCU_Module:WeMos_D1_mini U1
 U 1 1 63FB08E9
-P 1200 2700
-F 0 "U1" H 1550 1850 50  0000 C CNN
-F 1 "WeMos_D1_mini" H 1550 1950 50  0000 C CNN
-F 2 "Module:WEMOS_D1_mini_light" H 1200 1550 50  0001 C CNN
-F 3 "https://wiki.wemos.cc/products:d1:d1_mini#documentation" H -650 1550 50  0001 C CNN
-	1    1200 2700
+P 1200 3700
+F 0 "U1" H 1550 2850 50  0000 C CNN
+F 1 "WeMos_D1_mini" H 1550 2950 50  0000 C CNN
+F 2 "Module:WEMOS_D1_mini_light" H 1200 2550 50  0001 C CNN
+F 3 "https://wiki.wemos.cc/products:d1:d1_mini#documentation" H -650 2550 50  0001 C CNN
+	1    1200 3700
 	1    0    0    -1
 $EndComp
@@
 	1    0    0    -1
 $EndComp
-NoConn ~ 1600 2200
-Wire Wire Line
-	1600 2300 1650 2300
-Wire Wire Line
-	1650 2300 1650 1250
+NoConn ~ 1600 3200
+Wire Wire Line
+	1600 3300 1650 3300
 Wire Wire Line
 	1650 1250 3200 1250
 Wire Wire Line
-	1600 2500 1850 2500
-Wire Wire Line
-	1850 2500 1850 1650
-Wire Wire Line
-	1850 1650 3200 1650
-Wire Wire Line
-	1750 2400 1750 1350
+	1600 3500 1850 3500
 Wire Wire Line
 	1750 1350 3200 1350
 Wire Wire Line
-	1600 2400 1750 2400
+	1600 3400 1750 3400
 $Comp
 L power:+5V #PWR?
@@
 $EndComp
 Wire Wire Line
-	2600 750  3600 750
+	2600 750  3000 750
 Wire Wire Line
 	3600 750  3600 850
 Wire Wire Line
 	2600 750  1100 750
-Wire Wire Line
-	1100 750  1100 1900
 Connection ~ 2600 750
-NoConn ~ 800  2300
-NoConn ~ 800  2600
-NoConn ~ 800  2700
+NoConn ~ 800  3300
+NoConn ~ 800  3600
+NoConn ~ 800  3700
 Wire Wire Line
 	7500 6200 8450 6200
@@
 Wire Wire Line
 	4650 2650 6050 2650
-Wire Wire Line
-	1600 2800 4650 2800
-Wire Wire Line
-	4650 2800 4650 3800
-Wire Wire Line
-	4650 3800 6050 3800
-Wire Wire Line
-	1600 2900 4550 2900
-Wire Wire Line
-	4550 2900 4550 4850
-Wire Wire Line
-	4550 4850 6050 4850
-Wire Wire Line
-	1600 3000 4450 3000
-Wire Wire Line
-	4450 3000 4450 6000
-Wire Wire Line
-	4450 6000 6050 6000
 $Comp
 L power:GND #PWR?
@@
 L power:GND #PWR?
 U 1 1 640C9244
-P 1200 3900
-F 0 "#PWR?" H 1200 3650 50  0001 C CNN
-F 1 "GND" H 1205 3727 50  0000 C CNN
-F 2 "" H 1200 3900 50  0001 C CNN
-F 3 "" H 1200 3900 50  0001 C CNN
-	1    1200 3900
-	1    0    0    -1
-$EndComp
-Wire Wire Line
-	1200 3900 1200 3500
+P 1200 4900
+F 0 "#PWR?" H 1200 4650 50  0001 C CNN
+F 1 "GND" H 1205 4727 50  0000 C CNN
+F 2 "" H 1200 4900 50  0001 C CNN
+F 3 "" H 1200 4900 50  0001 C CNN
+	1    1200 4900
+	1    0    0    -1
+$EndComp
+Wire Wire Line
+	1200 4900 1200 4500
 Wire Wire Line
 	3600 2350 3600 2200
@@
 NoConn ~ 4000 1750
 NoConn ~ 4000 1950
-NoConn ~ 1600 3100
-NoConn ~ 1300 1900
+NoConn ~ 1600 4100
+NoConn ~ 1300 2900
 $Comp
 L Device:Fuse F1
@@
 Wire Wire Line
 	3600 2200 3600 2150
-NoConn ~ 3200 1050
 Connection ~ 5250 1050
 Wire Wire Line
@@
 	7500 6300 7500 6200
 Wire Wire Line
-	4650 2650 4650 2700
-Wire Wire Line
-	4650 2700 1600 2700
-Wire Wire Line
-	4550 1650 4550 2600
-Wire Wire Line
-	4550 2600 1600 2600
+	4650 3700 1600 3700
+Wire Wire Line
+	4550 3600 1600 3600
 Wire Wire Line
 	4550 1650 6050 1650
+Wire Wire Line
+	3000 750  3000 1650
+Wire Wire Line
+	3000 1650 3200 1650
+Connection ~ 3000 750
+Wire Wire Line
+	3000 750  3600 750
+Wire Wire Line
+	1850 1050 3200 1050
+Wire Wire Line
+	4550 4000 4550 6000
+Wire Wire Line
+	1600 3800 6050 3800
+Wire Wire Line
+	4650 2650 4650 3700
+Wire Wire Line
+	4550 1650 4550 3600
+Wire Wire Line
+	4650 4850 4650 3900
+Wire Wire Line
+	1600 4000 4550 4000
+Wire Wire Line
+	1600 3900 4650 3900
+Wire Wire Line
+	4650 4850 6050 4850
+Wire Wire Line
+	4550 6000 6050 6000
+Wire Wire Line
+	1850 1050 1850 3500
+Wire Wire Line
+	1750 1350 1750 3400
+Wire Wire Line
+	1650 1250 1650 3300
+Wire Wire Line
+	1100 750  1100 2900
 $EndSCHEMATC
